File: V1/ESP-pwm-4ch-V1.kicad_sch (KiCad schematic)
At the start: 32 parts, among them J1 12VDC, J2 OUT1, J3 OUT2, J4 OUT3, J5 OUT4, Q1 IRLB8721PBF, Q2 IRLB8721PBF, Q3 IRLB8721PBF, Q4 IRLB8721PBF, U1 L78M05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

Commit message: PCB tweaks
Other:
- title: ESP 6 PWM Module -> ESP 4 PWM Module
Changed lines of the file:
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@@
   (paper "A3")
   (title_block
-    (title "ESP 6 PWM Module")
+    (title "ESP 4 PWM Module")
     (date "2021-03-08")
     (rev "0.1")
